File: schematics/soft-starter.kicad_pcb (KiCad board)
At the start: 6 copper layers, 73 x 50 mm, 24 parts, among them J1 INPUT 12 V, J2 LED1, J3 LED2, J4 LED3, Q1 30N06, Q2 30N06, Q3 30N06, SW1 Reset, U1 ATtiny13-20P, U3 External DC-DC 5V

Commit message: Update pcb to actual thing
Parts:
- moved J2 10.2 mm to (134.6, 104.1)
- moved J4 5.08 mm to (134.6, 91.4)
- moved C1 4.39 mm to (121.9, 117.9)
- moved R1 2.54 mm to (106.7, 104.1)
- moved R2 2.54 mm to (106.7, 109.2)
- moved RV1 2.54 mm to (114.3, 114.3)
- moved RV2 2.54 mm to (109.2, 114.3)
- moved C2 2.12 mm to (104.1, 117.9), turned to -90 degrees
Routing:
- net GND: track 227.1 -> 188.5 mm
- net +12V: track 149.3 -> 159.7 mm
- net Net-(Q1-D): track 21.4 -> 12.7 mm
- net +5V: track 75.8 -> 68.2 mm
- net Net-(U1-PB2): track 44.2 -> 40.2 mm
- net Net-(Q3-D): track 16.3 -> 12.7 mm
- net Net-(Q2-D): track 16.3 -> 12.7 mm
- net Net-(Q1-G): track 7.62 -> 5.08 mm
- net Net-(U1-PB3): track 69.2 -> 67.4 mm
- net Net-(U1-PB4): track 37.7 -> 38.7 mm
Other:
- board text added: "LED0"
- board text added: "LED1"
- board text added: "LED2"
- board text added: "POT1"
- board text added: "POT2"
